File: Schematic/FBT.kicad_pcb (KiCad board)
At the start: 2 copper layers, 41.9 x 76.7 mm, 17 parts, among them J1 TRRS Connector 3.5, J5 Conn_01x04, SW2 SW_SPDT

Commit message: schematic work and notes
Parts:
- JP1: value 3v3 in -> 5v in
- JP2: value 5v in -> 3v3 in
- SW1: renamed from SW2; footprint My_Library:SS12F21 -> My_Library:SK12D07VG4
- moved D1 12.1 mm to (162.1, 65.8), turned to 90 degrees
- moved JP1 10.2 mm to (165.0, 69.0), turned to 180 degrees
- moved JP2 9.90 mm to (159.7, 77.5), turned to -90 degrees
- moved D2 8.51 mm to (162.1, 68.6), turned to 180 degrees
- moved REF** 7.00 mm to (143.8, 112.9), turned to -90 degrees
- moved GY2 3.97 mm to (162.6, 116.0)
- moved IMU2 3.97 mm to (162.6, 113.0)
- moved J2 3.97 mm to (165.6, 104.9)
- moved SW1 0.63 mm to (167.7, 62.2), turned to 90 degrees
- renumbered BT2 to BT1, U7 to CHGR1, D3 to D1, D4 to D2, U3 to GY1, U5 to GY2, U2 to IMU1, U4 to IMU2, J5 to J2, U1 to MCU1, R3 to R1, R4 to R2
Connections:
- D2 pad 2: Net-(D4-A) -> Net-(D2-A)
- GY1 pad 1: Net-(JP1-B) -> Net-(GY1-VIN)
- IMU1 pad 1: Net-(JP2-A) -> Net-(IMU1-VIN)
- IMU1 pad 2: Net-(JP1-B) -> Net-(GY1-VIN)
- JP1 pad 1: ESP32_3V3 -> Net-(IMU1-VIN)
- JP1 pad 2: Net-(JP1-B) -> ESP32_5V5
- JP2 pad 1: Net-(JP2-A) -> ESP32_3V3
- JP2 pad 2: ESP32_5V5 -> Net-(GY1-VIN)
- SW1 pad 1: Net-(D4-A) -> unconnected-(SW1-A-Pad1)
- SW1 pad 3: unconnected-(SW2-C-Pad3) -> Net-(D2-A)
Routing:
- net Net-(JP1-B): track 30.5 -> 0.00 mm, vias 2 -> 0
- net Net-(GY1-VIN): track 0.00 -> 29.2 mm, vias 0 -> 2
- net Net-(CHGR1-5_VIN): track 24.7 -> 3.37 mm
- net Net-(D2-A): track 0.00 -> 17.9 mm
- net ESP32_5V5: track 60.3 -> 43.7 mm, vias 2 -> 0
- net Net-(D4-A): track 13.3 -> 0.00 mm
- net SCL_1: track 52.4 -> 45.9 mm
- net +BATT: track 37.6 -> 43.6 mm
- net Net-(JP2-A): track 5.16 -> 0.00 mm
- net Net-(IMU1-VIN): track 0.00 -> 5.16 mm
- net ESP32_3V3: track 57.2 -> 55.7 mm
- net SDA_1: track 49.5 -> 48.1 mm
- net BATTERY_READER: vias 1 -> 0
Other:
- board size 41.9 x 76.7 mm -> 41.9 x 72.7 mm
