File: Schematic/Exports/MrTracker2/FBT.kicad_pcb (KiCad board)
At the start: 2 copper layers, 83.3 x 52 mm, 19 parts, among them J1 TRRS Connector 3.5, J2 TRRS Connector 3.5, SW1 SW_SPDT

Commit message: prep v2 PCB for production
Parts:
- removed GY2: ~, My_Library:GY-271
- removed IMU2: ~, My_Library:GY-BMI160
- removed J2: TRRS Connector 3.5, My_Library:PJ-320A
- removed the REF** at (176.5, 115.2)
Routing:
- net ESP32_3V3: track 62.0 -> 42.8 mm
- net SDA_1: track 63.1 -> 48.9 mm
- net GND: track 146.7 -> 134.1 mm
- net SCL_1: track 54.2 -> 45.9 mm
- net Net-(GY2-SDA): track 3.97 -> 0.00 mm
- net Net-(GY2-SCL): track 3.97 -> 0.00 mm
Other:
- board size 83.3 x 52 mm -> 40 x 40 mm
- board text removed: "UFBTM Type B Rev. 1.0"
