File: Schematic/Exports/MsTracker2/FBT.kicad_pcb (KiCad board)
At the start: 2 copper layers, 42.8 x 122.5 mm, 19 parts, among them J1 TRRS Connector 3.5, J2 TRRS Connector 3.5, SW1 SW_SPDT

Commit message: prep v2 PCB for production
Parts:
- removed GY2: ~, My_Library:GY-271
- removed IMU2: ~, My_Library:GY-BMI160
- removed J2: TRRS Connector 3.5, My_Library:PJ-320A
- removed REF**: GY-273, My_Library:GY-273
Routing:
- net ESP32_3V3: track 70.0 -> 50.9 mm
- net SDA_1: track 67.4 -> 53.3 mm
- net GND: track 135.7 -> 123.1 mm
- net SCL_1: track 61.1 -> 52.8 mm
- net Net-(GY2-SCL): track 3.97 -> 0.00 mm
- net Net-(GY2-SDA): track 3.97 -> 0.00 mm
Other:
- board size 42.8 x 122.5 mm -> 21 x 65.4 mm
- board text removed: "Type B Rev. 1.0"
