File: Schematic/Batt_804040/FBT.kicad_pcb (KiCad board)
At the start: 2 copper layers, 83.3 x 52 mm, 23 parts, among them J1 TRRS Connector 3.5, J2 TRRS Connector 3.5, SW1 SW_SPDT, U1 HT7333-1-TO92

Commit message: Work on documentation, fix Mr. Tracker Jumpers
The Rev 3.0 PCB unfortunately can't accommodate all regulator configs due to a mistake in the pin layout (forgetting which pins went where in the schematic)

This was resolved for Mr. Tracker
TODO: Mrs. Tracker
Parts:
- JP3: value A -> C
- JP4: value D -> A
- JP5: value B -> D
- JP6: value C -> B
- moved JP3 7.60 mm to (125.0, 126.0)
- moved JP4 7.55 mm to (132.5, 126.0), turned to 90 degrees
- moved JP5 2.60 mm to (127.5, 126.0)
- moved JP6 2.54 mm to (130.0, 126.0), turned to -90 degrees
Connections:
- net /gnd_mid renamed /vin_mid
- J1 pad R1: SDA_1 -> SCL_1
- J1 pad R2: SCL_1 -> GND
- J1 pad S: GND -> ESP32_3V3
- J1 pad T: ESP32_3V3 -> SDA_1
- J2 pad R1: SDA_1 -> SCL_1
- J2 pad R2: SCL_1 -> GND
- J2 pad S: GND -> ESP32_3V3
- J2 pad T: ESP32_3V3 -> SDA_1
- JP3 pad 2: /ldo_gnd -> /vin
- JP3 pad 3: BATT_SWITCHED -> ESP32_3V3
- JP4 pad 1: ESP32_3V3 -> GND
- JP4 pad 2: /vout -> /ldo_gnd
- JP4 pad 3: GND -> BATT_SWITCHED
- JP5 pad 1: BATT_SWITCHED -> ESP32_3V3
- JP5 pad 2: /vin -> /vout
- JP6 pad 1: GND -> BATT_SWITCHED
- JP6 pad 3: ESP32_3V3 -> GND
Routing:
- net /vout: track 13.6 -> 20.8 mm, vias 0 -> 1
- net /vin: track 19.8 -> 14.6 mm
- net GND: track 132.7 -> 137.2 mm
- net BATTERY_READER: track 34.4 -> 33.5 mm
